File: Quetta_hw/Quetta.kicad_pcb (KiCad board)
At the start: 2 copper layers, 87.5 x 42.4 mm, 83 parts, among them Q1 IRLML9303, Q2 BC817, SW1 SWITCH_H

Commit message: new pcb
Parts:
- removed C21, C22: 220pF, CAP_0603
- removed C34: 0.1u, CAP_0603
- removed XL5: USB_MICRO_B, USBmicro_MOLEX_WM17142
- added BLN1: BALUN868ST, Radio:BALUN868_ST, F.Cu at (136.2, 88.4)
- added C2: 10n, Capacitors:CAP_0603, F.Cu at (133.3, 120.4)
- added C4: 10n, Capacitors:CAP_0603, F.Cu at (138.8, 119.4)
- added C5: 1000u 6v3, Capacitors:CAP_08xxR, F.Cu at (131.2, 114.2)
- added C6: 18pF, Capacitors:CAP_0603, F.Cu at (143.7, 96.0)
- added C7: 18pF, Capacitors:CAP_0603, F.Cu at (143.7, 89.6)
- added C8: 0.1u, Capacitors:CAP_0603, F.Cu at (136.7, 97.2)
- added C9: 220pF, Capacitors:CAP_0603, F.Cu at (131.0, 90.0)
- added D2: SS14, Diodes:SMA_DO214AC, F.Cu at (135.4, 108.8)
- added L1: BLM15AG102SN1, Inductors:IND_0402, F.Cu at (131.7, 96.4)
- added L2: *, Inductors:IND_0402, F.Cu at (136.0, 84.3)
- added L3: BLM15AG102SN1, Inductors:IND_0402, F.Cu at (148.2, 94.3)
- added R14: 10k, Resistors:RES_0603, F.Cu at (132.9, 106.2)
- added R15: 56k, Resistors:RES_0603, F.Cu at (131.0, 91.5)
- added TP1: TESTPOINT, PCB:TESTPOINT_1MM, F.Cu at (139.9, 95.9)
- added XL2: USB_MINI_B, Connectors:USBmicro_MOLEX_WM17142, F.Cu at (140.1, 126.2)
- ANT1: value ANT_PCB_NOCNTR -> ANT_PCB_MONO; footprint ANT_FOLDED_DIPOLE2 -> Radio:ANT_868_45x18mm
- C1, C11, C12, C13, C17, C23, C24, C25, C27, C28, C29, C3, C31, C32, C33, C35, C36, C37, C38, C39, C40, C41, C42, C44, C45, C46, C47, C48, VCap1, VCap2: footprint CAP_0603 -> Capacitors:CAP_0603
- C10, C26, C30, C43: footprint CAP_0805 -> Capacitors:CAP_0805
- C14: value 220pF -> 10n; footprint CAP_0603 -> Capacitors:CAP_0603
- C15: value 0.1u -> 3.3pF; footprint CAP_0603 -> Capacitors:CAP_0603
- C16: value 0.1u -> 10n; footprint CAP_0603 -> Capacitors:CAP_0603
- C18: value 10pF -> 220pF; footprint CAP_0603 -> Capacitors:CAP_0603
- C19: value 10pF -> *; footprint CAP_0603 -> Capacitors:CAP_0402
- C20: value 0.1u -> *; footprint CAP_0603 -> Capacitors:CAP_0402
- D1: footprint LED0603 -> LEDs:LED_0603
- DA1: footprint LQFP48 -> LQFP_TQFP:LQFP48
- DA2: footprint DRB8 -> QFN_DFN:DRB8
- DA3: footprint SC82AB -> SOT:SC82AB
- DD1: footprint QFN16_5_3 -> QFN_DFN:QFN16_5_3
- DD2: value CC2500 -> CC1101; footprint QFN20 -> QFN_DFN:QFN20
- DD3: footprint LQFP64 -> LQFP_TQFP:LQFP64
- HOLE1, HOLE2, HOLE3, HOLE4: footprint Hole3_5_out6mm -> PCB:Hole3_5_out6mm
- Q1: footprint SOT23 -> SOT:SOT23-3
- Q2: value BC817 -> IRLML9303; footprint SOT23 -> SOT:SOT23-3
- R1, R10, R11, R12, R13, R2, R3, R5, R7, R8, R9: footprint RES_0603 -> Resistors:RES_0603
- R4: value 1k -> 1M; footprint RES_0603 -> Resistors:RES_0603
- R6: value 56k -> 20k; footprint RES_0603 -> Resistors:RES_0603
- SW1: footprint SW_SK12D07VG -> BtnsSwitches:SW_SS-1P2T
- XL1, XL11, XL3, XL7: footprint SIL-3 -> Connectors:PLS-3
- XL10: footprint SIL1_ROUND_1MM5 -> PCB:Round_1MM5
- XL4: footprint SIL-4 -> Connectors:PLS-4
- XL6: footprint SIL-2 -> Connectors:PLS-2
- XL8: footprint MICROSD_CAP_FIX05A -> Connectors:MICROSD_CAP_FIX05A
- XL9: footprint SIL1_SQUARE_1MM5 -> PCB:Square_1MM5
- XTAL1: footprint CRYSTAL_03225C4 -> Quartz:03225C4
- XTAL2: footprint CRYSTAL_0503x4-4 -> Quartz:0503x4-4
- moved R10 119.2 mm to (88.0, 136.0)
- moved R12 115.5 mm to (98.5, 136.0), turned to 0 degrees
- moved DA2 113.8 mm to (85.5, 98.0), turned to 0 degrees
- moved R13 112.1 mm to (103.5, 136.0), turned to 0 degrees
- moved C1 110.0 mm to (90.5, 81.5), turned to 0 degrees
- moved C10 108.4 mm to (90.0, 107.5), turned to 0 degrees
- moved C3 103.9 mm to (92.5, 97.0), turned to 0 degrees
- moved C19 100.4 mm to (136.5, 86.0), turned to 0 degrees
- moved C20 99.8 mm to (136.5, 82.6), turned to 0 degrees
- moved C14 98.2 mm to (134.4, 86.6)
- moved DD1 97.5 mm to (104.5, 104.0)
- moved C18 97.5 mm to (131.0, 93.0), turned to 180 degrees
- moved C15 97.2 mm to (139.8, 87.2), turned to 90 degrees
- moved HOLE3 97.0 mm to (130.3, 128.7)
- moved DD2 95.4 mm to (135.9, 91.8), turned to 90 degrees
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Connections:
- ANT1 pad 1: /Ant1 -> /ANT2
- C14 pad 1: +3.3V -> VCC
- C15 pad 1: +3.3V -> VCC
- C16 pad 1: +3.3V -> VCC
- C17 pad 1: N-0000020 -> VCC
- C18 pad 1: N-0000039 -> VCC
- C19 pad 1: N-0000040 -> /ANT1
- C20 pad 1: +3.3V -> /ANT2
- C23 pad 1: +3.3V -> /PWR_VS
- C24 pad 1: +3.3V -> /PWR_VS
- C25 pad 1: +3.3V -> /PWR_VS
- C26 pad 1: +3.3V -> /PWR_VS
- C27 pad 1: +3.3V -> /PWR_VS
- C28 pad 1: +3.3V -> /PWR_VS
- C29 pad 1: +3.3V -> /PWR_VS
- C30 pad 1: +3.3V -> /PWR_VS
- C33 pad 1: +BATT -> PwrUnst
- C47 pad 1: +BATT -> PwrUnst
- DA1 pad 14: +3.3V -> /PWR_VS
- DA1 pad 19: +3.3V -> /PWR_VS
- DA1 pad 32: +3.3V -> /PWR_VS
- DA1 pad 38: +3.3V -> /PWR_VS
- DA1 pad 43: +3.3V -> /PWR_VS
- DA1 pad 45: +3.3V -> /PWR_VS
- DA1 pad 6: +3.3V -> /PWR_VS
- DA2 pad 6: +BATT -> PwrUnst
- DA3 pad 1: +BATT -> PwrUnst
- DA3 pad 4: +BATT -> PwrUnst
- DD2 pad 10: N-0000040 -> Net-(C7-Pad1)
- DD2 pad 11: +3.3V -> VCC
- DD2 pad 12: /Ant1 -> /RF1
- DD2 pad 13: /Ant2 -> /RF2
- DD2 pad 14: +3.3V -> VCC
- DD2 pad 15: +3.3V -> VCC
- DD2 pad 17: N-0000017 -> Net-(DD2-Pad17)
- DD2 pad 18: N-0000023 -> VCC
- DD2 pad 4: +3.3V -> VCC
- DD2 pad 5: N-0000020 -> Net-(C8-Pad1)
- DD2 pad 8: N-0000039 -> Net-(C6-Pad1)
- DD2 pad 9: +3.3V -> VCC
- DD3 pad 44: /USB_DM -> /D-
- DD3 pad 45: /USB_DP -> /D+
- Q2 pad 1: N-0000046 -> +5V
- Q2 pad 2: GND -> PwrUnst
- Q2 pad 3: N-0000045 -> +BATT
- R13 pad 2: N-0000045 -> /BAT_MEASURE
- R4 pad 1: /BAT_MEASURE -> /SHLD
- R4 pad 2: N-0000046 -> GND
- R6 pad 1: N-0000017 -> /CC_CS
- R6 pad 2: GND -> VCC
- XTAL1 pad 1: N-0000039 -> Net-(C6-Pad1)
- XTAL1 pad 2: N-0000040 -> Net-(C7-Pad1)
Routing:
- net GND: track 502.0 -> 0.00 mm, vias 83 -> 0
- net +3.3V: track 244.8 -> 0.00 mm, vias 20 -> 0
- net +BATT: track 36.6 -> 0.00 mm, vias 1 -> 0
- net /SNS1_OUT: track 32.7 -> 0.00 mm, vias 1 -> 0
- net /TX2: track 31.7 -> 0.00 mm, vias 1 -> 0
- net /RX2: track 30.7 -> 0.00 mm, vias 1 -> 0
- net /AMPLF_SHDN: track 28.7 -> 0.00 mm, vias 2 -> 0
- net Net-(DD3-Pad2): track 25.5 -> 0.00 mm, vias 2 -> 0
- net /VS_DREQ: track 25.0 -> 0.00 mm, vias 2 -> 0
- net /CC_CS: track 23.7 -> 0.00 mm, vias 2 -> 0
- net /SNS2_OUT: track 22.5 -> 0.00 mm, vias 2 -> 0
- net /VS_SI: track 22.0 -> 0.00 mm, vias 2 -> 0
- net /VS_SO: track 21.0 -> 0.00 mm
- net /SND_L: track 20.8 -> 0.00 mm, vias 2 -> 0
- net /SD_CLK: track 20.7 -> 0.00 mm, vias 2 -> 0
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- removed copper zone on B.Cu, net GND
- removed copper zone on F.Cu, net GND
Other:
- board outline removed
- net class Default: trace_width 0.2 -> 0.25; via_dia 0.9 -> 0.6
- net class wide removed
- rule pad_to_mask_clearance: 0.075 -> 0.2
- rule via_min_drill: 0.4 -> 0.3
- rule via_min_size: 0.9 -> 0.4

Commit message: Components spreaded all over
Parts:
- removed XL7: CONN_3, Connectors:PLS-3
- C10, C26, C30, C43: footprint Capacitors:CAP_0805 -> Capacitors:CAP_0603
- XL4: value ST_SWD -> CONN_6; footprint Connectors:PLS-4 -> Connectors:PLS-6
- moved DA2 79.2 mm to (164.4, 90.8), turned to 270 degrees
- moved R2 74.5 mm to (131.0, 100.4), turned to 90 degrees
- moved R12 71.8 mm to (166.6, 113.4), turned to 270 degrees
- moved R8 71.2 mm to (163.2, 83.6), turned to 270 degrees
- moved R1 70.7 mm to (132.6, 100.4), turned to 270 degrees
- moved R10 70.1 mm to (152.8, 109.2), turned to 90 degrees
- moved C1 67.1 mm to (157.6, 83.0)
- moved R7 66.3 mm to (163.2, 86.6), turned to 90 degrees
- moved R5 66.2 mm to (160.0, 86.6), turned to 90 degrees
- moved R13 66.1 mm to (166.6, 116.4), turned to 270 degrees
- moved C3 65.8 mm to (157.6, 87.2)
- moved XL1 65.0 mm to (150.6, 130.6)
- moved R3 63.4 mm to (160.0, 83.6), turned to 270 degrees
- moved XL3 62.9 mm to (159.0, 130.6)
- moved XL11 57.4 mm to (159.0, 127.8)
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Connections:
- XL4 pad 1: +3.3V -> (no net)

Commit message: TopoR start
Other:
- net class Default: trace_width 0.25 -> 0.2; via_dia 0.6 -> 0.7; via_drill 0.4 -> 0.3
- net class Wide added: clearance 0.2, trace_width 0.5, via_dia 0.9, via_drill 0.4
Changed lines of the file:
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@@
     (links 265)
     (no_connects 265)
-    (area 0 0 0 0)
+    (area 125.86635 63.724999 172.275001 132.19057)
     (thickness 1.6)
     (drawings 3)
@@
   )
   (setup
-    (last_trace_width 0.25)
+    (last_trace_width 0.2)
     (trace_clearance 0.2)
     (zone_clearance 0.508)
@@
     (segment_width 0.2)
     (edge_width 0.15)
-    (via_size 0.6)
-    (via_drill 0.4)
+    (via_size 0.7)
+    (via_drill 0.3)
     (via_min_size 0.4)
     (via_min_drill 0.3)
@@
     (pad_to_mask_clearance 0.2)
     (aux_axis_origin 0 0)
-    (visible_elements 7FFFFF9F)
+    (visible_elements 7FFFF7BF)
     (pcbplotparams
       (layerselection 0x00030_80000001)
@@
   (net_class Default "This is the default net class."
     (clearance 0.2)
-    (trace_width 0.25)
-    (via_dia 0.6)
-    (via_drill 0.4)
+    (trace_width 0.2)
+    (via_dia 0.7)
+    (via_drill 0.3)
     (uvia_dia 0.3)
     (uvia_drill 0.1)
-    (add_net +3.3V)
-    (add_net +5V)
-    (add_net +BATT)
     (add_net /12MHz_Clk)
     (add_net /ACC_IRQ)
@@
     (add_net /ANT1)
     (add_net /ANT2)
-    (add_net /BATTERY_PLUS)
     (add_net /BAT_MEASURE)
     (add_net /CC_CS)
@@
     (add_net /VS_XCS)
     (add_net /VS_XDCS)
-    (add_net GND)
     (add_net "Net-(C1-Pad2)")
     (add_net "Net-(C12-Pad1)")
@@
     (add_net "Net-(DD3-Pad47)")
     (add_net "Net-(DD3-Pad6)")
+  )
+  (net_class Wide ""
+    (clearance 0.2)
+    (trace_width 0.5)
+    (via_dia 0.9)
+    (via_drill 0.4)
+    (uvia_dia 0.3)
+    (uvia_drill 0.1)
+    (add_net +3.3V)
+    (add_net +5V)
+    (add_net +BATT)
+    (add_net /BATTERY_PLUS)
+    (add_net GND)
     (add_net PwrUnst)
     (add_net VCC)

Commit message: Gerber done
Parts:
- moved C43 15.8 mm to (146.8, 100.1), turned to 90 degrees
- moved C36 8.41 mm to (157.4, 113.2), turned to 180 degrees
- moved C37 7.63 mm to (157.4, 105.2), turned to 0 degrees
- moved C46 2.02 mm to (152.6, 114.6)
- moved C23 1.61 mm to (160.2, 92.4)
- moved TP1 1.61 mm to (138.3, 96.2)
- moved C13 1.59 mm to (160.2, 94.0)
- moved C44 1.06 mm to (152.4, 105.2)
- moved C45 1.06 mm to (154.0, 105.2)
- moved C42 0.93 mm to (148.4, 100.1), turned to 90 degrees
- moved R10 0.82 mm to (153.3, 109.9)
- moved XTAL2 0.41 mm to (157.1, 109.2), turned to 90 degrees
- moved C35 0.13 mm to (159.9, 90.1)
Routing:
- net GND: track 0.00 -> 598.8 mm, vias 0 -> 176
- net +3.3V: track 0.00 -> 142.3 mm, vias 0 -> 5
- net VCC: track 0.00 -> 60.7 mm, vias 0 -> 4
- net /PWR_VS: track 0.00 -> 60.3 mm, vias 0 -> 4
- net Net-(DD3-Pad2): track 0.00 -> 46.7 mm, vias 0 -> 2
- net /AMPLF_SHDN: track 0.00 -> 39.1 mm, vias 0 -> 4
- net PwrUnst: track 0.00 -> 35.7 mm
- net /I2C_SDA: track 0.00 -> 32.0 mm, vias 0 -> 4
- net /SNS3_OUT: track 0.00 -> 31.8 mm, vias 0 -> 1
- net /D-: track 0.00 -> 30.4 mm, vias 0 -> 2
- net /D+: track 0.00 -> 30.2 mm, vias 0 -> 2
- net /SNS2_OUT: track 0.00 -> 30.0 mm, vias 0 -> 1
- net /ACC_IRQ: track 0.00 -> 29.5 mm, vias 0 -> 2
- net /VS_RST: track 0.00 -> 28.4 mm, vias 0 -> 2
- net /I2C_SCL: track 0.00 -> 28.2 mm, vias 0 -> 4
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- added copper zone on B.Cu, net GND
- added copper zone on F.Cu, net GND
Other:
- board outline added: 45 x 68 mm
- rule pad_to_mask_clearance: 0.2 -> 0.1

Commit message: + Ostranna logo * Vias now all 0.3 drill + Gerbers sent to production
Parts:
- added Logo1: Logo, Pictures:Ostranna_16d9_13d5, F.Cu at (160.2, 73.2)
Other:
- net class Wide: via_drill 0.4 -> 0.3
- board text added: "Quetta HW2"
