File: Quetta_hw/Quetta.kicad_pcb (KiCad board)
At the start: 4 copper layers, 54 x 36 mm, 122 parts, among them Q1 IRLML6401, Q2 IRLML6401, Q3 IRLML6401, Q4 IRLML6401

Commit message: + Gerbers sent to factory
Parts:
- moved Logo1 77.4 mm to (287.9, 111.0)
Routing:
- net GND: track 396.4 -> 316.9 mm, vias 115 -> 120
- added copper zone on B.Cu, net /+5V_USB
- added copper zone on In1.Cu, net /+5V_USB
- added copper zone on In2.Cu, net /+5V_USB
- added copper zone on B.Cu, net /+AU_PWR
Other:
- board text added: "+"
- board text added: "+3v3"
- board text added: "ANT"
- board text added: "Charger"
- board text added: "DATA"
- board text added: "GND"
- board text added: "Neopixel"
- board text added: "Ostranna Quetta3"
- board text added: "PA0"
- board text added: "PA1"
- board text added: "PA8"
- board text added: "PB1"
- board text added: "PC0"
- board text added: "PC1"
- board text added: "PWR"
- board text added: "Radio"
- board text added: "Speaker"
- board text removed: "Ostranna Flute2"
