File: Quetta_hw/Quetta.sch (KiCad schematic (older format))
At the start: 83 parts, among them Q1 IRLML9303, Q2 BC817, SW1 SWITCH_H

Commit message: + Quetta HW2
Parts:
- removed ANT1: ANT_PCB_NOCNTR, ~, symbol ANT_PCB_NOCNTR
- removed C21, C22: 220pF, symbol C
- removed C34: 0.1u, CAP_0402, symbol C
- removed DD2: CC2500, symbol CC2500
- removed Q2: BC817, ~, symbol NPN
- removed XL5: USB_MICRO_B, symbol USB_MINI_B
- added ANT1: ANT_PCB_MONO, Radio:ANT_868_MEANDER_4HOR_35mm, symbol ANT_PCB_MONO
- added BLN1: BALUN868ST, symbol BALUN868ST
- added C2, C4: 10n, Capacitors:CAP_0603, symbol C
- added C5: 1000u 6v3, symbol CP
- added C6, C7: 18pF, Capacitors:CAP_0603, symbol C
- added C8: 0.1u, Capacitors:CAP_0603, symbol C
- added C9: 220pF, Capacitors:CAP_0603, symbol C
- added D2: SS14, symbol D_Shottky
- added DD2: CC1101, QFN:QFN20, symbol CC1101
- added L1, L3: BLM15AG102SN1, Inductors:IND_0402, symbol L
- added L2: *, Inductors:IND_0402, symbol L
- added Q2: IRLML9303, SOT:SOT23-3, symbol IRLML6302
- added R14: 10k, Resistors:RES_0603, symbol R
- added R15: 56k, Resistors:RES_0603, symbol R
- added TP1: TESTPOINT, PCB:TESTPOINT_1MM, symbol TESTPOINT
- added XL2: USB_MINI_B, Connectors:USBmicro_MOLEX_WM17142, symbol USB_MINI_B
- C13, C23, C24, C25, C27, C28, C29: footprint CAP_0603 -> (none)
- C14: value 220pF -> 10n; footprint (none) -> Capacitors:CAP_0603
- C15: value 0.1u -> 3.3pF; footprint (none) -> Capacitors:CAP_0603
- C16: value 0.1u -> 10n; footprint (none) -> Capacitors:CAP_0603
- C17: footprint (none) -> Capacitors:CAP_0603
- C18: value 10pF -> 220pF; footprint CAP_0402 -> Capacitors:CAP_0603
- C19: value 10pF -> *; footprint CAP_0402 -> Capacitors:CAP_0402
- C20: value 0.1u -> *; footprint (none) -> Capacitors:CAP_0402
- C26, C30, C43: footprint CAP_0805 -> (none)
- C36, C37, C39, C40, C41, C42, C44, C45, C46, VCap1, VCap2: footprint CAP_0402 -> (none)
- D1, DD3, SW1, XL1, XL11, XL3: footprint ~ -> (none)
- R10, R9: footprint RES_0402 -> (none)
- R11: footprint RES_0603 -> (none)
- R4: value 1k -> 1M; footprint RES_0603 -> Resistors:RES_0603
- R6: value 56k -> 20k; footprint (none) -> Resistors:RES_0603
- XTAL1: footprint 03225 -> Quartz:03225C4
- XTAL2: footprint 0532 -> (none)
Connections:
- net labels added: ANT1, ANT2, D+, D-, PWR_VS, PwrUnst, RF1, RF2, SHLD, VCC
- net labels removed: Ant1, Ant2, USB_DM, USB_DP
- wire segments 280 -> 309
Other:
- note added: "5v OR Battery\nauto switch"
- note added: "Balun"
- note added: "CC Power Filter"
- note added: "Keep CS High\nwhen sleeping"
- note added: "Matching circuit"
- note added: "Pins 15, 14, 11, 9, 4, 18"
- moved on the sheet: C47, C48, DA3, R12, R13, XL10, XL9

Commit message: Components choosen
Parts:
- ANT1: footprint Radio:ANT_868_MEANDER_4HOR_35mm -> Radio:ANT_868_45x18mm
- BLN1: footprint (none) -> Radio:BALUN868_ST
- C1, C11, C12, C13, C23, C24, C25, C27, C28, C29, C3, C31, C32, C33, C35, C36, C37, C38, C39, C40, C41, C42, C44, C45, C46, C47, C48, VCap1, VCap2: footprint (none) -> Capacitors:CAP_0603
- C10, C26, C30, C43: footprint (none) -> Capacitors:CAP_0805
- C5: footprint (none) -> Capacitors:CAP_08xxR
- D1: footprint (none) -> LEDs:LED_0603
- D2: footprint (none) -> Diodes:SMA_DO214AC
- DA1: footprint (none) -> LQFP_TQFP:LQFP48
- DA2: footprint (none) -> QFN_DFN:DRB8
- DA3: footprint (none) -> SOT:SC82AB
- DD1: footprint (none) -> QFN_DFN:QFN16_5_3
- DD3: footprint (none) -> LQFP_TQFP:LQFP64
- HOLE1, HOLE2, HOLE3, HOLE4: footprint (none) -> PCB:Hole3_5_out6mm
- Q1: footprint (none) -> SOT:SOT23-3
- R1, R10, R11, R12, R13, R2, R3, R5, R7, R8, R9: footprint (none) -> Resistors:RES_0603
- SW1: footprint (none) -> BtnsSwitches:SW_SS-1P2T
- XL1, XL11, XL3, XL7: footprint (none) -> Connectors:PLS-3
- XL10: footprint (none) -> Connectors:Round_1MM5
- XL4: footprint (none) -> Connectors:PLS-4
- XL6: footprint (none) -> Connectors:PLS-2
- XL8: footprint (none) -> Connectors:MICROSD_CAP_FIX05A; URL (none) -> http://www.zip-2002.ru/razyemy/derzhateli_sim_i_kart_pamyat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
- XL9: footprint (none) -> Connectors:Square_1MM5
- XTAL2: footprint (none) -> Quartz:0503x4-4

Commit message: new pcb
Parts:
- DD2: footprint QFN:QFN20 -> QFN_DFN:QFN20
- XL10: footprint Connectors:Round_1MM5 -> PCB:Round_1MM5
- XL9: footprint Connectors:Square_1MM5 -> PCB:Square_1MM5
Changed lines of the file:
@@
 F 0 "XL10" V 2850 15210 40  0000 C CNN
 F 1 "CONN_1" V 2910 15220 40  0000 C CNN
-F 2 "Connectors:Round_1MM5" H 2900 15200 60  0001 C CNN
+F 2 "PCB:Round_1MM5" H 2900 15200 60  0001 C CNN
 F 3 "" H 2900 15200 60  0001 C CNN
 	1    2900 15200
@@
 F 0 "XL9" V 2850 14760 40  0000 C CNN
 F 1 "CONN_1" V 2910 14770 40  0000 C CNN
-F 2 "Connectors:Square_1MM5" H 2900 14750 60  0001 C CNN
+F 2 "PCB:Square_1MM5" H 2900 14750 60  0001 C CNN
 F 3 "" H 2900 14750 60  0001 C CNN
 	1    2900 14750
@@
 F 0 "DD2" H 7500 3000 60  0000 C CNN
 F 1 "CC1101" H 8250 3000 60  0000 C CNN
-F 2 "QFN:QFN20" H 7950 2200 60  0001 C CNN
+F 2 "QFN_DFN:QFN20" H 7950 2200 60  0001 C CNN
 F 3 "" H 7950 2200 60  0001 C CNN
 	1    7950 2200

Commit message: Components spreaded all over
Parts:
- removed XL4: ST_SWD, Connectors:PLS-4, symbol ST_SWD
- removed XL7: CONN_3, Connectors:PLS-3, symbol CONN_3
- added XL4: CONN_6, Connectors:PLS-6, symbol CONN_6
- C10, C26, C30, C43: footprint Capacitors:CAP_0805 -> Capacitors:CAP_0603
- TP1: symbol TESTPOINT -> TESTPOINT-RESCUE-Quetta
Connections:
- net GND: now also XL4.3
- net RX2: now also XL4.6
- net SWCLK: now also XL4.2
- net SWDIO: now also XL4.4
- net TX2: now also XL4.5
- new net PwrMCU: XL4.1
Other:
- note removed: "DEBUG \nTX/RX"

Commit message: + Ostranna logo * Vias now all 0.3 drill + Gerbers sent to production
Parts:
- added Logo1: Logo, Pictures:Ostranna_16d9_13d5, symbol Logo
Changed lines of the file:
@@
 Wire Wire Line
 	12150 7450 12850 7450
+$Comp
+L Logo Logo1
+U 1 1 571695D2
+P 19250 10000
+F 0 "Logo1" H 19150 10450 60  0000 C CNN
+F 1 "Logo" H 19450 10450 60  0000 C CNN
+F 2 "Pictures:Ostranna_16d9_13d5" H 19250 10000 60  0001 C CNN
+F 3 "" H 19250 10000 60  0000 C CNN
+	1    19250 10000
+	1    0    0    -1
+$EndComp
 $EndSCHEMATC
